File: hardware/SMB/PS-SegmentMonitoringBoard.kicad_pcb (KiCad board)
At the start: 4 copper layers, 89 x 85 mm, 126 parts, among them IC1 BQ79616PAPR, J1 voltTapConn, J2 highSideConn, J3 lowSideConn, J4 thermConn, Q1 ZXTN4004KTC

Commit message: ss fixes
Other:
- board text added: "High Side"
- board text added: "Low Side"
- board text added: "X"
- board text removed: "High Side Conn"
- board text removed: "Low Side Conn"
Changed lines of the file:
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@@
 		(layer "F.SilkS")
 	)
-	(gr_line
-		(start 126.05 131.1)
-		(end 125.33 131.82)
-		(stroke
-			(width 0.1)
-			(type default)
-		)
-		(layer "F.SilkS")
-	)
-	(gr_line
-		(start 126.05 131.1)
-		(end 127.84 131.1)
-		(stroke
-			(width 0.1)
-			(type default)
-		)
-		(layer "F.SilkS")
-	)
 	(gr_rect
 		(start 127.425 75.175)
@@
 		)
 	)
+	(gr_text "X\n"
+		(at 83.83 84.46 0)
+		(layer "F.SilkS")
+		(effects
+			(font
+				(size 1 1)
+				(thickness 0.2)
+			)
+			(justify left bottom)
+		)
+	)
 	(gr_text "V0"
 		(at 84.49 120.27 0)
@@
 	)
 	(gr_text "LN"
-		(at 114.93 132.94 0)
+		(at 115.05 132.93 0)
 		(layer "F.SilkS")
 		(effects
@@
 	)
 	(gr_text "HN"
-		(at 117.85 132.98 0)
+		(at 117.83 133 0)
 		(layer "F.SilkS")
 		(effects
@@
 	)
 	(gr_text "HP"
-		(at 127.89 132.28 0)
+		(at 127.9 133.04 0)
 		(layer "F.SilkS")
 		(effects
@@
 		)
 	)
+	(gr_text "X"
+		(at 130.79 133.06 0)
+		(layer "F.SilkS")
+		(effects
+			(font
+				(size 1 1)
+				(thickness 0.2)
+			)
+			(justify left bottom)
+		)
+	)
 	(gr_text "T0"
 		(at 145.66 80.84 0)
@@
 		)
 	)
-	(gr_text "Cell Volts & Balancing"
-		(at 88.77 113.4 0)
+	(gr_text "Low Side"
+		(at 109.06 142.66 90)
 		(layer "F.SilkS")
 		(effects
 			(font
 				(size 1 1)
-				(thickness 2)
+				(thickness 0.25)
 			)
 			(justify left bottom)
 		)
 	)
-	(gr_text "LDOIN BJT"
-		(at 130.79 111.34 0)
+	(gr_text "High Side"
+		(at 130.59 142.73 90)
 		(layer "F.SilkS")
 		(effects
 			(font
 				(size 1 1)
-				(thickness 2)
+				(thickness 0.25)
 			)
 			(justify left bottom)
 		)
 	)
-	(gr_text "Thermistors"
-		(at 136.17 76.95 0)
+	(gr_text "Cell Volts & Balancing"
+		(at 88.77 113.4 0)
 		(layer "F.SilkS")
 		(effects
@@
 		)
 	)
-	(gr_text "Low Side Conn\n"
-		(at 107 143.09 90)
+	(gr_text "LDOIN BJT"
+		(at 130.79 111.34 0)
 		(layer "F.SilkS")
 		(effects
@@
 		)
 	)
-	(gr_text "Isolation"
-		(at 130.88 122.15 90)
+	(gr_text "Thermistors"
+		(at 136.17 76.95 0)
 		(layer "F.SilkS")
 		(effects
@@
 		)
 	)
-	(gr_text "High Side Conn\n"
-		(at 131.91 143.18 90)
+	(gr_text "Isolation"
+		(at 130.88 122.15 90)
 		(layer "F.SilkS")
 		(effects
