File: hardware/SMB/Cell_Balancing.kicad_sch (KiCad schematic)
At the start: 16 parts

Commit message: added cell tap 9
Parts:
- added C21: 0.47uF, Capacitor_SMD:C_0603_1608Metric_Pad1.08x0.95mm_HandSolder, symbol Device:C_Small
- added R67: 6.2, Resistor_SMD:R_2512_6332Metric_Pad1.40x3.35mm_HandSolder, symbol Device:R_Small
Connections:
- net CB7: now also C21.2; no longer C13.2
- new net CB8: C13.2, C21.1, R67.2
- new net V8: R67.1
Other:
- moved on the sheet: C13

Commit message: added BOM
Parts:
- C13, C14, C15, C16, C17, C18, C19, C20, C21: value 0.47uF -> 0.47u; P/N (none) -> CC0603KRX7R7BB474
- R10, R11, R4, R5, R6, R67, R7, R8, R9: P/N (none) -> ERJ-1TRQF6R2U
Changed lines of the file:
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@@
+			)
+		)
+		(property "P/N" "ERJ-1TRQF6R2U"
+			(at 95.25 53.34 90)
+			(hide yes)
+			(show_name no)
+			(do_not_autoplace no)
+			(effects
+				(font
+					(size 1.27 1.27)
+				)
 			)
 		)
@@
 			)
 		)
-		(property "Value" "0.47uF"
+		(property "Value" "0.47u"
 			(at 110.49 42.164 0)
 			(show_name no)
@@
 			)
 		)
+		(property "P/N" "CC0603KRX7R7BB474"
+			(at 110.49 40.64 0)
+			(hide yes)
+			(show_name no)
+			(do_not_autoplace no)
+			(effects
+				(font
+					(size 1.27 1.27)
+				)
+			)
+		)
 		(pin "1"
 		)
@@
 			)
 		)
-		(property "Value" "0.47uF"
+		(property "Value" "0.47u"
 			(at 110.49 72.644 0)
 			(show_name no)
@@
 		)
 		(property "Description" "Unpolarized capacitor, small symbol"
+			(at 110.49 71.12 0)
+			(hide yes)
+			(show_name no)
+			(do_not_autoplace no)
+			(effects
+				(font
+					(size 1.27 1.27)
+				)
+			)
+		)
+		(property "P/N" "CC0603KRX7R7BB474"
 			(at 110.49 71.12 0)
 			(hide yes)
@@
 			)
 		)
+		(property "P/N" "ERJ-1TRQF6R2U"
+			(at 95.25 63.5 90)
+			(hide yes)
+			(show_name no)
+			(do_not_autoplace no)
+			(effects
+				(font
+					(size 1.27 1.27)
+				)
+			)
+		)
 		(pin "2"
 		)
@@
 			)
 		)
+		(property "P/N" "ERJ-1TRQF6R2U"
+			(at 95.25 48.26 90)
+			(hide yes)
+			(show_name no)
+			(do_not_autoplace no)
+			(effects
+				(font
+					(size 1.27 1.27)
+				)
+			)
+		)
 		(pin "2"
 		)
@@
 			)
 		)
-		(property "Value" "0.47uF"
+		(property "Value" "0.47u"
 			(at 110.49 67.564 0)
 			(show_name no)
@@
 		)
 		(property "Description" "Unpolarized capacitor, small symbol"
+			(at 110.49 66.04 0)
+			(hide yes)
+			(show_name no)
+			(do_not_autoplace no)
+			(effects
+				(font
+					(size 1.27 1.27)
+				)
+			)
+		)
+		(property "P/N" "CC0603KRX7R7BB474"
 			(at 110.49 66.04 0)
 			(hide yes)
@@
 			)
 		)
+		(property "P/N" "ERJ-1TRQF6R2U"
+			(at 95.25 43.18 90)
+			(hide yes)
+			(show_name no)
+			(do_not_autoplace no)
+			(effects
+				(font
+					(size 1.27 1.27)
+				)
+			)
+		)
 		(pin "2"
 		)
@@
 			)
 		)
-		(property "Value" "0.47uF"
+		(property "Value" "0.47u"
 			(at 110.49 47.244 0)
 			(show_name no)
@@
 		)
 		(property "Description" "Unpolarized capacitor, small symbol"
+			(at 110.49 45.72 0)
+			(hide yes)
+			(show_name no)
+			(do_not_autoplace no)
+			(effects
+				(font
+					(size 1.27 1.27)
+				)
+			)
+		)
+		(property "P/N" "CC0603KRX7R7BB474"
 			(at 110.49 45.72 0)
 			(hide yes)
@@
 			)
 		)
+		(property "P/N" "ERJ-1TRQF6R2U"
+			(at 95.25 58.42 90)
+			(hide yes)
+			(show_name no)
+			(do_not_autoplace no)
+			(effects
+				(font
+					(size 1.27 1.27)
+				)
+			)
+		)
 		(pin "2"
 		)
@@
 			)
 		)
-		(property "Value" "0.47uF"
+		(property "Value" "0.47u"
 			(at 110.49 32.004 0)
 			(show_name no)
@@
 		)
 		(property "Description" "Unpolarized capacitor, small symbol"
+			(at 110.49 30.48 0)
+			(hide yes)
+			(show_name no)
+			(do_not_autoplace no)
+			(effects
+				(font
+					(size 1.27 1.27)
+				)
+			)
+		)
+		(property "P/N" "CC0603KRX7R7BB474"
 			(at 110.49 30.48 0)
 			(hide yes)
@@
 			)
 		)
+		(property "P/N" "ERJ-1TRQF6R2U"
+			(at 95.25 73.66 90)
+			(hide yes)
+			(show_name no)
+			(do_not_autoplace no)
+			(effects
+				(font
+					(size 1.27 1.27)
+				)
+			)
+		)
 		(pin "2"
 		)
@@
 			)
 		)
-		(property "Value" "0.47uF"
+		(property "Value" "0.47u"
 			(at 110.49 37.084 0)
 			(show_name no)
@@
 			)
 		)
+		(property "P/N" "CC0603KRX7R7BB474"
+			(at 110.49 35.56 0)
+			(hide yes)
+			(show_name no)
+			(do_not_autoplace no)
+			(effects
+				(font
+					(size 1.27 1.27)
+				)
+			)
+		)
 		(pin "1"
 		)
@@
 			)
 		)
-		(property "Value" "0.47uF"
+		(property "Value" "0.47u"
 			(at 110.49 52.324 0)
 			(show_name no)
@@
 		)
 		(property "Description" "Unpolarized capacitor, small symbol"
+			(at 110.49 50.8 0)
+			(hide yes)
+			(show_name no)
+			(do_not_autoplace no)
+			(effects
+				(font
+					(size 1.27 1.27)
+				)
+			)
+		)
+		(property "P/N" "CC0603KRX7R7BB474"
 			(at 110.49 50.8 0)
 			(hide yes)
@@
 			)
 		)
+		(property "P/N" "ERJ-1TRQF6R2U"
+			(at 95.25 33.02 90)
+			(hide yes)
+			(show_name no)
+			(do_not_autoplace no)
+			(effects
+				(font
+					(size 1.27 1.27)
+				)
+			)
+		)
 		(pin "2"
 		)
@@
 			)
 		)
-		(property "Value" "0.47uF"
+		(property "Value" "0.47u"
 			(at 110.49 57.404 0)
 			(show_name no)
@@
 		)
 		(property "Description" "Unpolarized capacitor, small symbol"
+			(at 110.49 55.88 0)
+			(hide yes)
+			(show_name no)
+			(do_not_autoplace no)
+			(effects
+				(font
+					(size 1.27 1.27)
+				)
+			)
+		)
+		(property "P/N" "CC0603KRX7R7BB474"
 			(at 110.49 55.88 0)
 			(hide yes)
@@
 			)
 		)
+		(property "P/N" "ERJ-1TRQF6R2U"
+			(at 95.25 38.1 90)
+			(hide yes)
+			(show_name no)
+			(do_not_autoplace no)
+			(effects
+				(font
+					(size 1.27 1.27)
+				)
+			)
+		)
 		(pin "2"
 		)
@@
 			)
 		)
+		(property "P/N" "ERJ-1TRQF6R2U"
+			(at 95.25 68.58 90)
+			(hide yes)
+			(show_name no)
+			(do_not_autoplace no)
+			(effects
+				(font
+					(size 1.27 1.27)
+				)
+			)
+		)
 		(pin "2"
 		)
@@
 			)
 		)
-		(property "Value" "0.47uF"
+		(property "Value" "0.47u"
 			(at 110.49 62.484 0)
 			(show_name no)
@@
 			(at 110.49 60.96 0)
 			(hide yes)
+			(show_name no)
+			(do_not_autoplace no)
+			(effects
+				(font
+					(size 1.27 1.27)
+				)
+			)
+		)
+		(property "P/N" "CC0603KRX7R7BB474"
+			(at 110.49 60.96 0)
+			(hide yes)
