File: hardware/SMB/PS-SegmentMonitoringBoard.kicad_sch (KiCad schematic)
At the start: 21 parts, among them IC1 BQ79616PAPR, J1 voltTapsConn, J2 highSideConn, J3 lowSideConn, J4 thermsConn

Commit message: added cell tap 9
Parts:
- removed J1: voltTapsConn, LHRS_Connectors:Molex_Nano-Fit_105313-xx08_1x08_P2.50mm_Horizontal, symbol Connector_Generic:Conn_01x08
- added J1: voltTapConn, Custom-Footprints:1053141110, symbol Connector_Generic:Conn_01x10
Connections:
- net V0: now also J1.9 (Pin_9)
- net V1: now also J1.8 (Pin_8)
- net V2: now also J1.7 (Pin_7)
- net V3: now also J1.6 (Pin_6)
- net V4: now also J1.5 (Pin_5)
- net V5: now also J1.4 (Pin_4)
- net V6: now also J1.3 (Pin_3)
- net V7: now also J1.2 (Pin_2)
- net extraCells: no longer IC1.18 (CB8), IC1.19 (VC8)
- new net CB8: IC1.18 (CB8)
- new net V8: J1.1 (Pin_1)
- new net VC8: IC1.19 (VC8)
- no-connect marks 5 -> 6

Commit message: added ntcs gnda
Parts:
- removed J4: thermsConn, LHRS_Connectors:Molex_Nano-Fit_105313-xx08_1x08_P2.50mm_Horizontal, symbol Connector_Generic:Conn_01x08
- added J4: thermConn, Custom-Footprints:1053141116, symbol Connector_Generic:Conn_01x16
Connections:
- net AVSS: now also J4.10 (Pin_10), J4.11 (Pin_11), J4.12 (Pin_12), J4.13 (Pin_13), J4.14 (Pin_14), J4.15 (Pin_15), J4.16 (Pin_16), J4.9 (Pin_9)
- net TEMP_0: now also J4.8 (Pin_8)
- net TEMP_1: now also J4.7 (Pin_7)
- net TEMP_2: now also J4.6 (Pin_6)
- net TEMP_3: now also J4.5 (Pin_5)
- net TEMP_4: now also J4.4 (Pin_4)
- net TEMP_5: now also J4.3 (Pin_3)
- net TEMP_6: now also J4.2 (Pin_2)
- net TEMP_7: now also J4.1 (Pin_1)

Commit message: added BOM
Parts:
- C1: value 1uF -> 1u; P/N (none) -> CC0603KRX7R9BB105
- C2: value 1uF -> 1u; P/N (none) -> GRM21BR61H106KE43L
- C3: value 22nF -> 22n; P/N (none) -> CC0603KRX7R9BB223
- C4: value 4.7uF -> 4.7u; P/N (none) -> 06035C472K4T2A
- C5: value 100nF -> 100n; P/N (none) -> CL10B104KB8NNNC
- C6: P/N (none) -> CC0603KRX7R7BB225
- C7: value 0.1uF -> 0.1u; P/N (none) -> CL10B104KB8NNNC
- IC1: Height 1.2 -> (none); Manufacturer_Name Texas Instruments -> (none); Manufacturer_Part_Number BQ79616PAPR -> (none); Mouser Part Number 595-BQ79616PAPR -> (none); Mouser Price/Stock https://www.mouser.co.uk/ProductDetail/Texas-Instruments/BQ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 -> (none); P/N (none) -> BQ79616PAPR
Changed lines of the file:
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@@
 			)
 		)
-		(property "Value" "22nF"
+		(property "Value" "22n"
 			(at 71.628 76.708 0)
 			(show_name no)
@@
 		)
 		(property "Description" "Unpolarized capacitor, small symbol"
+			(at 68.58 74.93 0)
+			(hide yes)
+			(show_name no)
+			(do_not_autoplace no)
+			(effects
+				(font
+					(size 1.27 1.27)
+				)
+			)
+		)
+		(property "P/N" "CC0603KRX7R9BB223"
 			(at 68.58 74.93 0)
 			(hide yes)
@@
 			)
 		)
-		(property "PN" ""
-			(at 265.43 160.02 0)
-			(hide yes)
-			(show_name no)
-			(do_not_autoplace no)
-			(effects
-				(font
-					(size 1.27 1.27)
-				)
-			)
-		)
-		(property "p/n" ""
-			(at 265.43 160.02 0)
-			(hide yes)
-			(show_name no)
-			(do_not_autoplace no)
-			(effects
-				(font
-					(size 1.27 1.27)
-				)
-			)
-		)
 		(instances
 			(project "PS-SegmentMonitoringBoard"
@@
 			)
 		)
-		(property "Value" "1uF"
+		(property "Value" "1u"
 			(at 62.992 76.708 0)
 			(show_name no)
@@
 		)
 		(property "Description" "Unpolarized capacitor, small symbol"
+			(at 60.96 74.93 0)
+			(hide yes)
+			(show_name no)
+			(do_not_autoplace no)
+			(effects
+				(font
+					(size 1.27 1.27)
+				)
+			)
+		)
+		(property "P/N" "GRM21BR61H106KE43L"
 			(at 60.96 74.93 0)
 			(hide yes)
@@
 			)
 		)
-		(property "Value" "4.7uF"
+		(property "Value" "4.7u"
 			(at 80.518 76.708 0)
 			(show_name no)
@@
 		)
 		(property "Description" "Unpolarized capacitor, small symbol"
+			(at 77.47 74.93 0)
+			(hide yes)
+			(show_name no)
+			(do_not_autoplace no)
+			(effects
+				(font
+					(size 1.27 1.27)
+				)
+			)
+		)
+		(property "P/N" "06035C472K4T2A"
 			(at 77.47 74.93 0)
 			(hide yes)
@@
 			)
 		)
-		(property "Height" "1.2"
-			(at 175.26 413.97 0)
-			(hide yes)
-			(show_name no)
-			(do_not_autoplace no)
-			(effects
-				(font
-					(size 1.27 1.27)
-				)
-				(justify left top)
-			)
-		)
-		(property "Mouser Part Number" "595-BQ79616PAPR"
-			(at 175.26 513.97 0)
-			(hide yes)
-			(show_name no)
-			(do_not_autoplace no)
-			(effects
-				(font
-					(size 1.27 1.27)
-				)
-				(justify left top)
-			)
-		)
-		(property "Mouser Price/Stock" "https://www.mouser.co.uk/ProductDetail/Texas-Instruments/BQ79616PAPR?qs=1Kr7Jg1SGW8FUVDCFv5r0A%3D%3D"
-			(at 175.26 613.97 0)
-			(hide yes)
-			(show_name no)
-			(do_not_autoplace no)
-			(effects
-				(font
-					(size 1.27 1.27)
-				)
-				(justify left top)
-			)
-		)
-		(property "Manufacturer_Name" "Texas Instruments"
-			(at 175.26 713.97 0)
-			(hide yes)
-			(show_name no)
-			(do_not_autoplace no)
-			(effects
-				(font
-					(size 1.27 1.27)
-				)
-				(justify left top)
-			)
-		)
-		(property "Manufacturer_Part_Number" "BQ79616PAPR"
-			(at 175.26 813.97 0)
-			(hide yes)
-			(show_name no)
-			(do_not_autoplace no)
-			(effects
-				(font
-					(size 1.27 1.27)
-				)
-				(justify left top)
+		(property "P/N" "BQ79616PAPR"
+			(at 123.19 29.21 0)
+			(hide yes)
+			(show_name no)
+			(do_not_autoplace no)
+			(effects
+				(font
+					(size 1.27 1.27)
+				)
 			)
 		)
@@
 			)
 		)
-		(property "Value" "100nF"
+		(property "Value" "100n"
 			(at 89.408 76.708 0)
 			(show_name no)
@@
 		)
 		(property "Description" "Unpolarized capacitor, small symbol"
+			(at 86.36 74.93 0)
+			(hide yes)
+			(show_name no)
+			(do_not_autoplace no)
+			(effects
+				(font
+					(size 1.27 1.27)
+				)
+			)
+		)
+		(property "P/N" "CL10B104KB8NNNC"
 			(at 86.36 74.93 0)
 			(hide yes)
@@
 			)
 		)
+		(property "P/N" "CC0603KRX7R7BB225"
+			(at 93.98 74.93 0)
+			(hide yes)
+			(show_name no)
+			(do_not_autoplace no)
+			(effects
+				(font
+					(size 1.27 1.27)
+				)
+			)
+		)
 		(pin "2"
 		)
@@
 			)
 		)
-		(property "Value" "0.1uF"
+		(property "Value" "0.1u"
 			(at 116.586 40.64 90)
 			(show_name no)
@@
 		(property "Description" "Unpolarized capacitor, small symbol"
 			(at 113.03 39.37 0)
+			(hide yes)
+			(show_name no)
+			(do_not_autoplace no)
+			(effects
+				(font
+					(size 1.27 1.27)
+				)
+			)
+		)
+		(property "P/N" "CL10B104KB8NNNC"
+			(at 113.03 39.37 90)
 			(hide yes)
 			(show_name no)
@@
 			)
 		)
-		(property "Value" "1uF"
+		(property "Value" "1u"
 			(at 55.372 76.708 0)
 			(show_name no)
@@
 			(at 53.34 74.93 0)
 			(hide yes)
+			(show_name no)
+			(do_not_autoplace no)
+			(effects
+				(font
+					(size 1.27 1.27)
+				)
+			)
+		)
+		(property "P/N" "CC0603KRX7R9BB105"
+			(at 53.34 74.93 0)
+			(hide yes)
