File: hardware/SMB/Thermistors.kicad_sch (KiCad schematic)
At the start: 49 parts

Commit message: added BOM
Parts:
- C29, C30, C31, C32, C33, C34, C35, C36, C37: value 1uF -> 1u; P/N (none) -> GRM21BR61H106KE43L
- R17, R18, R19, R20, R21, R22, R23, R24: P/N (none) -> 0603WAF1001T5E
- R25, R26, R27, R28, R29, R30, R31, R32: P/N (none) -> CRCW060315K0FKEA
- R33, R34, R35, R36, R37, R38, R39, R40: P/N (none) -> RC0603FR-133K6L
- R41, R42, R43, R44, R45, R46, R47, R48: P/N (none) -> 0603WAF1003T5E
- R49, R50, R51, R52, R53, R54, R55, R56: P/N (none) -> 0603WAF1002T5E
