File: hardware/SMB/Volt_Taps.kicad_sch (KiCad schematic)
At the start: 18 parts

Commit message: added cell tap 9
Parts:
- added C47: 0.47uF, Capacitor_SMD:C_0603_1608Metric_Pad1.08x0.95mm_HandSolder, symbol Device:C_Small
- added R66: 100, Resistor_SMD:R_0603_1608Metric_Pad0.98x0.95mm_HandSolder, symbol Device:R_Small
Connections:
- net V7: no longer R57.2
- net VC7: now also C47.2
- new net V8: R57.2, R66.1
- new net VC8: C47.1, R66.2
Other:
- moved on the sheet: C38, R57

Commit message: added BOM
Parts:
- C38: value 10nF -> 10n; P/N (none) -> GCM188R71H103KA37J
- C39, C40, C41, C42, C43, C44, C45, C46, C47: value 0.47uF -> 0.47u; P/N (none) -> CC0603KRX7R7BB474
- R57: P/N (none) -> RC0603FR-0730RL
- R58, R59, R60, R61, R62, R63, R64, R65, R66: P/N (none) -> 0603WAF1000T5E
Changed lines of the file:
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@@
+			)
+		)
+		(property "P/N" "0603WAF1000T5E"
+			(at 55.88 64.77 90)
+			(hide yes)
+			(show_name no)
+			(do_not_autoplace no)
+			(effects
+				(font
+					(size 1.27 1.27)
+				)
 			)
 		)
@@
 			)
 		)
+		(property "P/N" "0603WAF1000T5E"
+			(at 55.88 80.01 90)
+			(hide yes)
+			(show_name no)
+			(do_not_autoplace no)
+			(effects
+				(font
+					(size 1.27 1.27)
+				)
+			)
+		)
 		(pin "2"
 		)
@@
 			)
 		)
-		(property "Value" "0.47uF"
+		(property "Value" "0.47u"
 			(at 76.708 50.546 0)
 			(show_name no)
@@
 			)
 		)
+		(property "P/N" "CC0603KRX7R7BB474"
+			(at 69.85 52.07 0)
+			(hide yes)
+			(show_name no)
+			(do_not_autoplace no)
+			(effects
+				(font
+					(size 1.27 1.27)
+				)
+			)
+		)
 		(pin "1"
 		)
@@
 			)
 		)
+		(property "P/N" "0603WAF1000T5E"
+			(at 55.88 59.69 90)
+			(hide yes)
+			(show_name no)
+			(do_not_autoplace no)
+			(effects
+				(font
+					(size 1.27 1.27)
+				)
+			)
+		)
 		(pin "2"
 		)
@@
 			)
 		)
+		(property "P/N" "0603WAF1000T5E"
+			(at 55.88 54.61 90)
+			(hide yes)
+			(show_name no)
+			(do_not_autoplace no)
+			(effects
+				(font
+					(size 1.27 1.27)
+				)
+			)
+		)
 		(pin "2"
 		)
@@
 			)
 		)
-		(property "Value" "0.47uF"
+		(property "Value" "0.47u"
 			(at 76.708 86.106 0)
 			(show_name no)
@@
 			)
 		)
+		(property "P/N" "CC0603KRX7R7BB474"
+			(at 69.85 87.63 0)
+			(hide yes)
+			(show_name no)
+			(do_not_autoplace no)
+			(effects
+				(font
+					(size 1.27 1.27)
+				)
+			)
+		)
 		(pin "1"
 		)
@@
 			)
 		)
+		(property "P/N" "0603WAF1000T5E"
+			(at 55.88 44.45 90)
+			(hide yes)
+			(show_name no)
+			(do_not_autoplace no)
+			(effects
+				(font
+					(size 1.27 1.27)
+				)
+			)
+		)
 		(pin "2"
 		)
@@
 			)
 		)
+		(property "P/N" "0603WAF1000T5E"
+			(at 55.88 49.53 90)
+			(hide yes)
+			(show_name no)
+			(do_not_autoplace no)
+			(effects
+				(font
+					(size 1.27 1.27)
+				)
+			)
+		)
 		(pin "2"
 		)
@@
 			)
 		)
-		(property "Value" "0.47uF"
+		(property "Value" "0.47u"
 			(at 76.708 60.706 0)
 			(show_name no)
@@
 			)
 		)
+		(property "P/N" "CC0603KRX7R7BB474"
+			(at 69.85 62.23 0)
+			(hide yes)
+			(show_name no)
+			(do_not_autoplace no)
+			(effects
+				(font
+					(size 1.27 1.27)
+				)
+			)
+		)
 		(pin "1"
 		)
@@
 			)
 		)
+		(property "P/N" "0603WAF1000T5E"
+			(at 55.88 74.93 90)
+			(hide yes)
+			(show_name no)
+			(do_not_autoplace no)
+			(effects
+				(font
+					(size 1.27 1.27)
+				)
+			)
+		)
 		(pin "2"
 		)
@@
 			)
 		)
-		(property "Value" "0.47uF"
+		(property "Value" "0.47u"
 			(at 76.708 55.626 0)
 			(show_name no)
@@
 			)
 		)
+		(property "P/N" "CC0603KRX7R7BB474"
+			(at 69.85 57.15 0)
+			(hide yes)
+			(show_name no)
+			(do_not_autoplace no)
+			(effects
+				(font
+					(size 1.27 1.27)
+				)
+			)
+		)
 		(pin "1"
 		)
@@
 			)
 		)
-		(property "Value" "0.47uF"
+		(property "Value" "0.47u"
 			(at 76.708 81.026 0)
 			(show_name no)
@@
 			)
 		)
+		(property "P/N" "CC0603KRX7R7BB474"
+			(at 69.85 82.55 0)
+			(hide yes)
+			(show_name no)
+			(do_not_autoplace no)
+			(effects
+				(font
+					(size 1.27 1.27)
+				)
+			)
+		)
 		(pin "1"
 		)
@@
 			)
 		)
+		(property "P/N" "0603WAF1000T5E"
+			(at 55.88 69.85 90)
+			(hide yes)
+			(show_name no)
+			(do_not_autoplace no)
+			(effects
+				(font
+					(size 1.27 1.27)
+				)
+			)
+		)
 		(pin "2"
 		)
@@
 			)
 		)
+		(property "P/N" "0603WAF1000T5E"
+			(at 55.88 85.09 90)
+			(hide yes)
+			(show_name no)
+			(do_not_autoplace no)
+			(effects
+				(font
+					(size 1.27 1.27)
+				)
+			)
+		)
 		(pin "2"
 		)
@@
 			)
 		)
-		(property "Value" "0.47uF"
+		(property "Value" "0.47u"
 			(at 76.708 75.946 0)
 			(show_name no)
@@
 			)
 		)
+		(property "P/N" "CC0603KRX7R7BB474"
+			(at 69.85 77.47 0)
+			(hide yes)
+			(show_name no)
+			(do_not_autoplace no)
+			(effects
+				(font
+					(size 1.27 1.27)
+				)
+			)
+		)
 		(pin "1"
 		)
@@
 			)
 		)
-		(property "Value" "0.47uF"
+		(property "Value" "0.47u"
 			(at 76.708 65.786 0)
 			(show_name no)
@@
 			)
 		)
+		(property "P/N" "CC0603KRX7R7BB474"
+			(at 69.85 67.31 0)
+			(hide yes)
+			(show_name no)
+			(do_not_autoplace no)
+			(effects
+				(font
+					(size 1.27 1.27)
+				)
+			)
+		)
 		(pin "1"
 		)
@@
 			)
 		)
-		(property "Value" "10nF"
+		(property "Value" "10n"
 			(at 69.85 25.146 0)
 			(show_name no)
@@
 		)
 		(property "Description" "Unpolarized capacitor, small symbol"
+			(at 69.85 26.67 0)
+			(hide yes)
+			(show_name no)
+			(do_not_autoplace no)
+			(effects
+				(font
+					(size 1.27 1.27)
+				)
+			)
+		)
+		(property "P/N" "GCM188R71H103KA37J"
 			(at 69.85 26.67 0)
 			(hide yes)
@@
 			)
 		)
+		(property "P/N" "RC0603FR-0730RL"
+			(at 55.88 22.86 90)
+			(hide yes)
+			(show_name no)
+			(do_not_autoplace no)
+			(effects
+				(font
+					(size 1.27 1.27)
+				)
+			)
+		)
 		(pin "2"
 		)
@@
 			)
 		)
-		(property "Value" "0.47uF"
+		(property "Value" "0.47u"
 			(at 76.708 70.866 0)
 			(show_name no)
@@
 			)
 		)
+		(property "P/N" "CC0603KRX7R7BB474"
+			(at 69.85 72.39 0)
+			(hide yes)
+			(show_name no)
+			(do_not_autoplace no)
+			(effects
+				(font
+					(size 1.27 1.27)
+				)
+			)
+		)
 		(pin "1"
 		)
@@
 			)
 		)
-		(property "Value" "0.47uF"
+		(property "Value" "0.47u"
 			(at 76.708 45.466 0)
 			(show_name no)
@@
 			(at 69.85 46.99 0)
 			(hide yes)
+			(show_name no)
+			(do_not_autoplace no)
+			(effects
+				(font
+					(size 1.27 1.27)
+				)
+			)
+		)
+		(property "P/N" "CC0603KRX7R7BB474"
+			(at 69.85 46.99 0)
+			(hide yes)
